Commit message: stl name update

File: bmkbot_description/urdf/bmkbot_gazebo.urdf.xacro (robot description, xacro)
@@ -12,5 +12,5 @@
             <origin xyz="0 0 0" rpy="0 0 0"/>
             <geometry>
-            <mesh filename="file://$(find bmkbot_description)/meshes/bmkbotbot/base_link.stl" scale="0.001 0.001 0.001"/>
+            <mesh filename="file://$(find bmkbot_description)/meshes/bmkbot/base_link.stl" scale="0.001 0.001 0.001"/>
             </geometry>
             <material name="silver"/>
@@ -19,5 +19,5 @@
             <origin xyz="0 0 0" rpy="0 0 0"/>
             <geometry>
-            <mesh filename="file://$(find bmkbot_description)/meshes/bmkbotbot/base_link.stl" scale="0.001 0.001 0.001"/>
+            <mesh filename="file://$(find bmkbot_description)/meshes/bmkbot/base_link.stl" scale="0.001 0.001 0.001"/>
             </geometry>
         </collision>
@@ -52,5 +52,5 @@
             <origin xyz="-0.157776 -0.085 -0.03" rpy="0 0 0"/>
             <geometry>
-            <mesh filename="file://$(find bmkbot_description)/meshes/bmkbotbot/wheel_right_1.stl" scale="0.001 0.001 0.001"/>
+            <mesh filename="file://$(find bmkbot_description)/meshes/bmkbot/wheel_right.stl" scale="0.001 0.001 0.001"/>
             </geometry>
             <material name="silver"/>
@@ -59,5 +59,5 @@
             <origin xyz="-0.157776 -0.085 -0.03" rpy="0 0 0"/>
             <geometry>
-            <mesh filename="file://$(find bmkbot_description)/meshes/bmkbotbot/wheel_right_1.stl" scale="0.001 0.001 0.001"/>
+            <mesh filename="file://$(find bmkbot_description)/meshes/bmkbot/wheel_right.stl" scale="0.001 0.001 0.001"/>
             </geometry>
         </collision>
@@ -72,5 +72,5 @@
             <origin xyz="0.157224 -0.085 -0.03" rpy="0 0 0"/>
             <geometry>
-            <mesh filename="file://$(find bmkbot_description)/meshes/bmkbotbot/wheel_left_1.stl" scale="0.001 0.001 0.001"/>
+            <mesh filename="file://$(find bmkbot_description)/meshes/bmkbot/wheel_left.stl" scale="0.001 0.001 0.001"/>
             </geometry>
             <material name="silver"/>
@@ -79,5 +79,5 @@
             <origin xyz="0.157224 -0.085 -0.03" rpy="0 0 0"/>
             <geometry>
-            <mesh filename="file://$(find bmkbot_description)/meshes/bmkbotbot/wheel_left_1.stl" scale="0.001 0.001 0.001"/>
+            <mesh filename="file://$(find bmkbot_description)/meshes/bmkbot/wheel_left.stl" scale="0.001 0.001 0.001"/>
             </geometry>
         </collision>
@@ -92,5 +92,5 @@
             <origin xyz="0.25 0.0 -0.273" rpy="0 0 -1.57"/>
             <geometry>
-            <mesh filename="file://$(find bmkbot_description)/meshes/bmkbotbot/camera_link_1.stl" scale="0.001 0.001 0.001"/>
+            <mesh filename="file://$(find bmkbot_description)/meshes/bmkbot/camera_link.stl" scale="0.001 0.001 0.001"/>
             </geometry>
             <material name="silver"/>
@@ -99,5 +99,5 @@
             <origin xyz="-0.0 0.245 -0.273" rpy="0 0 0"/>
             <geometry>
-            <mesh filename="file://$(find bmkbot_description)/meshes/bmkbotbot/camera_link_1.stl" scale="0.001 0.001 0.001"/>
+            <mesh filename="file://$(find bmkbot_description)/meshes/bmkbot/camera_link.stl" scale="0.001 0.001 0.001"/>
             </geometry>
         </collision>
@@ -112,5 +112,5 @@
             <origin xyz="-0.0 -0.0 -0.205" rpy="0 0 0"/>
             <geometry>
-            <mesh filename="file://$(find bmkbot_description)/meshes/bmkbotbot/lidar_link_1.stl" scale="0.001 0.001 0.001"/>
+            <mesh filename="file://$(find bmkbot_description)/meshes/bmkbot/lidar_link.stl" scale="0.001 0.001 0.001"/>
             </geometry>
             <material name="silver"/>
@@ -119,5 +119,5 @@
             <origin xyz="-0.0 -0.0 -0.205" rpy="0 0 0"/>
             <geometry>
-            <mesh filename="file://$(find bmkbot_description)/meshes/bmkbotbot/lidar_link_1.stl" scale="0.001 0.001 0.001"/>
+            <mesh filename="file://$(find bmkbot_description)/meshes/bmkbot/lidar_link.stl" scale="0.001 0.001 0.001"/>
             </geometry>
         </collision>
@@ -132,5 +132,5 @@
             <origin xyz="-0.0 0.194 -0.0" rpy="0 0 0"/>
             <geometry>
-            <mesh filename="file://$(find bmkbot_description)/meshes/bmkbotbot/ballcaster_link_1.stl" scale="0.001 0.001 0.001"/>
+            <mesh filename="file://$(find bmkbot_description)/meshes/bmkbot/ballcaster_link.stl" scale="0.001 0.001 0.001"/>
             </geometry>
             <material name="silver"/>
@@ -139,5 +139,5 @@
             <origin xyz="-0.0 0.194 -0.0" rpy="0 0 0"/>
             <geometry>
-            <mesh filename="file://$(find bmkbot_description)/meshes/bmkbotbot/ballcaster_link_1.stl" scale="0.001 0.001 0.001"/>
+            <mesh filename="file://$(find bmkbot_description)/meshes/bmkbot/ballcaster_link.stl" scale="0.001 0.001 0.001"/>
             </geometry>
         </collision>
@@ -181,4 +181,4 @@
         <child link="caster_link"/>
     </joint>
-    <xacro:include filename="$(find bmkbot_description)/gazebo/bmkbotbot.gazebo.xacro" />
+    <xacro:include filename="$(find bmkbot_description)/gazebo/bmkbot.gazebo.xacro" />
 </robot>
